File: hw2/PIC32_board/board.sch (EAGLE design)
At the start: 22 parts, among them J1 USB-MB-H

Commit message: Complete board design, add PCB gerber files.
Parts:
- removed V_REG(3.3V): MCP1702, me433:MCP1702
- added U$1: SOT-223, me433:SOT-223
- C1: device me433:CPOL-USCT6032 -> me433:CAP-POL; SPICEPREFIX C -> (none)
- C2, C3, C4, C7: device rcl:C-USC1206 -> resistor:C-USC0603
- C5: device me433:CPOL-USCT6032 -> me433:CAP-POL
- CLOCK: value OSCO -> OSC; device me433:OSCO -> me433:OSC
- GREEN: value (none) -> GREEN; device led:LED3MM -> me433:LED-GREEN0603
- J1: value USB-MB-H -> USB; device me433:USB-MB-H -> me433:USB
- R1, R2, R3, R4: device resistor:R-US_R1206 -> resistor:R-US_R0603
- RED: value (none) -> RED; device led:LED3MM -> me433:LED-RED0603
Connections:
- net N$3 renamed VCAP
- net N$7 renamed OSC2
- net N$8 renamed OSC1
- removed net PGD\: PIC.4.PGED1
- net +3V3: now also U$1.2.VOUT; no longer V_REG(3.3V).3.VOUT
- net +5V: now also U$1.3.VIN, U$1.4.VOUT; no longer V_REG(3.3V).2.VIN
- net GND: now also PIC.8.VSS, U$1.1.GND; no longer V_REG(3.3V).1.GND
- net PGD: now also PIC.4.PGED1
Other:
- moved on the sheet: C2, R1
