File: hw2/PIC32_board/lcd.sch (EAGLE design)
At the start: 1 part

Commit message: Add IMU schematic and README info
Parts:
- added IMU: LSM6DS33, me433:LSM6DS33
Connections:
- new net SCL2/RB3: IMU.5.SCL
- new net SDA2/RB2: IMU.4.SDA
- net +3V3: now also IMU.1.VDD, IMU.2.VIN
- net GND: now also IMU.3.GND
Changed lines of the file:
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@@
 <part name="+3V2" library="me433" deviceset="+3V3" device=""/>
 <part name="+3V3" library="me433" deviceset="+3V3" device=""/>
+<part name="IMU" library="me433" deviceset="LSM6DS33" device=""/>
+<part name="GND2" library="me433" deviceset="GND" device=""/>
+<part name="+3V4" library="me433" deviceset="+3V3" device=""/>
 </parts>
 <sheets>
@@
 </segment>
 </net>
+</nets>
+</sheet>
+<sheet>
+<plain>
+</plain>
+<instances>
+<instance part="IMU" gate="G$1" x="0" y="0"/>
+<instance part="GND2" gate="1" x="-15.24" y="7.62"/>
+<instance part="+3V4" gate="G$1" x="-15.24" y="22.86"/>
+</instances>
+<busses>
+</busses>
+<nets>
+<net name="+3V3" class="0">
+<segment>
+<pinref part="IMU" gate="G$1" pin="2.VIN"/>
+<pinref part="+3V4" gate="G$1" pin="+3V3"/>
+<wire x1="-12.7" y1="12.7" x2="-15.24" y2="12.7" width="0.1524" layer="91"/>
+<wire x1="-15.24" y1="12.7" x2="-15.24" y2="17.78" width="0.1524" layer="91"/>
+<pinref part="IMU" gate="G$1" pin="1.VDD"/>
+<wire x1="-15.24" y1="17.78" x2="-15.24" y2="20.32" width="0.1524" layer="91"/>
+<wire x1="-12.7" y1="17.78" x2="-15.24" y2="17.78" width="0.1524" layer="91"/>
+<junction x="-15.24" y="17.78"/>
+</segment>
+</net>
+<net name="GND" class="0">
+<segment>
+<pinref part="GND2" gate="1" pin="GND"/>
+<pinref part="IMU" gate="G$1" pin="3.GND"/>
+<wire x1="-15.24" y1="10.16" x2="-12.7" y2="7.62" width="0.1524" layer="91"/>
+</segment>
+</net>
+<net name="SDA2/RB2" class="0">
+<segment>
+<pinref part="IMU" gate="G$1" pin="4.SDA"/>
+<wire x1="-12.7" y1="2.54" x2="-27.94" y2="2.54" width="0.1524" layer="91"/>
+<label x="-27.94" y="2.54" size="1.778" layer="95"/>
+</segment>
+</net>
+<net name="SCL2/RB3" class="0">
+<segment>
+<pinref part="IMU" gate="G$1" pin="5.SCL"/>
+<wire x1="-12.7" y1="-2.54" x2="-27.94" y2="-2.54" width="0.1524" layer="91"/>
+<label x="-27.94" y="-2.54" size="1.778" layer="95"/>
+</segment>
+</net>
